File: transmitter/hardware/transmitter/transmitter.sch (KiCad schematic (older format))
At the start: 29 parts, among them J1 SOIL, J2 SOIL, J3 USB_UART_OFF, J4 USB_UART_ON, J5 SOIL, J6 SOIL, J7 SOIL, J8 SOIL, SW1 SW_SPST, U1 NodeMCU_1.0_(ESP-12E)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

Commit message: Vin & battery straps
Parts:
- removed H3, H4: MountingHole, MountingHole:MountingHole_3.2mm_M3_Pad, symbol Mechanical:MountingHole_Pad
- added F1: Polyfuse, Fuse:Fuse_1812_4532Metric_Pad1.30x3.40mm_HandSolder, symbol Device:Polyfuse_Small
- added SW2: SW, Connector_PinHeader_2.54mm:PinHeader_1x02_P2.54mm_Vertical, symbol Switch:SW_SPST
Connections:
- wire segments 55 -> 57
- no-connect marks 17 -> 16
Other:
- moved on the sheet: C3, C4, U2
Changed lines of the file:
@@
 L power:GND #PWR06
 U 1 1 5DBC1A3A
-P 2225 3125
-F 0 "#PWR06" H 2225 2875 50  0001 C CNN
-F 1 "GND" H 2230 2952 50  0000 C CNN
-F 2 "" H 2225 3125 50  0001 C CNN
-F 3 "" H 2225 3125 50  0001 C CNN
-	1    2225 3125
+P 2625 3125
+F 0 "#PWR06" H 2625 2875 50  0001 C CNN
+F 1 "GND" H 2630 2952 50  0000 C CNN
+F 2 "" H 2625 3125 50  0001 C CNN
+F 3 "" H 2625 3125 50  0001 C CNN
+	1    2625 3125
 	1    0    0    -1
 $EndComp
@@
 L Regulator_Linear:MCP1700-3302E_SOT89 U2
 U 1 1 5DBC1D4F
-P 2225 2600
-F 0 "U2" H 2225 2842 50  0000 C CNN
-F 1 "MCP1700-3302E_SOT89" H 2225 2751 50  0000 C CNN
-F 2 "Package_TO_SOT_SMD:SOT-89-3" H 2225 2800 50  0001 C CNN
-F 3 "http://ww1.microchip.com/downloads/en/DeviceDoc/20001826C.pdf" H 2225 2550 50  0001 C CNN
-	1    2225 2600
+P 2625 2600
+F 0 "U2" H 2625 2842 50  0000 C CNN
+F 1 "MCP1700-3302E_SOT89" H 2625 2751 50  0000 C CNN
+F 2 "Package_TO_SOT_SMD:SOT-89-3" H 2625 2800 50  0001 C CNN
+F 3 "http://ww1.microchip.com/downloads/en/DeviceDoc/20001826C.pdf" H 2625 2550 50  0001 C CNN
+	1    2625 2600
 	1    0    0    -1
 $EndComp
@@
 L Device:C_Small C3
 U 1 1 5DBC2404
-P 1475 2800
-F 0 "C3" H 1567 2846 50  0000 L CNN
-F 1 "1uF" H 1567 2755 50  0000 L CNN
-F 2 "Capacitor_SMD:C_0603_1608Metric_Pad1.05x0.95mm_HandSolder" H 1475 2800 50  0001 C CNN
-F 3 "~" H 1475 2800 50  0001 C CNN
-	1    1475 2800
+P 2050 2800
+F 0 "C3" H 2142 2846 50  0000 L CNN
+F 1 "1uF" H 2142 2755 50  0000 L CNN
+F 2 "Capacitor_SMD:C_0603_1608Metric_Pad1.05x0.95mm_HandSolder" H 2050 2800 50  0001 C CNN
+F 3 "~" H 2050 2800 50  0001 C CNN
+	1    2050 2800
 	1    0    0    -1
 $EndComp
@@
 L Device:C_Small C4
 U 1 1 5DBC2493
-P 2950 2800
-F 0 "C4" H 3042 2846 50  0000 L CNN
-F 1 "1uF" H 3042 2755 50  0000 L CNN
-F 2 "Capacitor_SMD:C_0603_1608Metric_Pad1.05x0.95mm_HandSolder" H 2950 2800 50  0001 C CNN
-F 3 "~" H 2950 2800 50  0001 C CNN
-	1    2950 2800
+P 3350 2800
+F 0 "C4" H 3442 2846 50  0000 L CNN
+F 1 "1uF" H 3442 2755 50  0000 L CNN
+F 2 "Capacitor_SMD:C_0603_1608Metric_Pad1.05x0.95mm_HandSolder" H 3350 2800 50  0001 C CNN
+F 3 "~" H 3350 2800 50  0001 C CNN
+	1    3350 2800
 	1    0    0    -1
 $EndComp
 Wire Wire Line
-	2950 2700 2950 2600
+	3350 2700 3350 2600
 Wire Wire Line
-	2950 2600 2525 2600
+	3350 2600 2925 2600
 Wire Wire Line
-	875  2600 1475 2600
+	2050 2700 2050 2600
 Wire Wire Line
-	1475 2700 1475 2600
-Connection ~ 1475 2600
+	2050 2900 2625 2900
 Wire Wire Line
-	1475 2600 1925 2600
+	3350 2900 2625 2900
+Connection ~ 2625 2900
 Wire Wire Line
-	1475 2900 2225 2900
-Wire Wire Line
-	2950 2900 2225 2900
-Connection ~ 2225 2900
-Wire Wire Line
-	2225 2900 2225 3050
+	2625 2900 2625 3050
 Wire Wire Line
 	875  3000 875  3050
 Wire Wire Line
-	875  3050 2225 3050
-Connection ~ 2225 3050
+	875  3050 2625 3050
+Connection ~ 2625 3050
 Wire Wire Line
-	2225 3050 2225 3125
-Text Label 1125 2600 0    50   ~ 0
+	2625 3050 2625 3125
+Text Label 1825 2600 0    50   ~ 0
 BATT
 NoConn ~ 6025 4425
@@
 3V3
 Wire Wire Line
-	2950 2600 3525 2600
-Connection ~ 2950 2600
+	3350 2600 3525 2600
+Connection ~ 3350 2600
 Text GLabel 6025 4325 0    50   Input ~ 0
 3V3
@@
 Text Notes 650  700  0    79   ~ 16
 Sensors
-NoConn ~ 6025 4725
 $Comp
 L Connector_Generic:Conn_01x01 J3
@@
 	1    0    0    -1
 $EndComp
+NoConn ~ 9875 5025
+Text Label 5825 4725 0    50   ~ 0
+BATT
+Wire Wire Line
+	6025 4725 5825 4725
 $Comp
-L Mechanical:MountingHole_Pad H3
-U 1 1 5DBE5750
-P 2400 4150
-F 0 "H3" H 2500 4201 50  0000 L CNN
-F 1 "MountingHole" H 2200 4325 50  0000 L CNN
-F 2 "MountingHole:MountingHole_3.2mm_M3_Pad" H 2400 4150 50  0001 C CNN
-F 3 "~" H 2400 4150 50  0001 C CNN
-	1    2400 4150
-	1    0    0    -1
-$EndComp
-$Comp
-L power:GND #PWR018
-U 1 1 5DBE5756
-P 2400 4250
-F 0 "#PWR018" H 2400 4000 50  0001 C CNN
-F 1 "GND" H 2405 4077 50  0000 C CNN
-F 2 "" H 2400 4250 50  0001 C CNN
-F 3 "" H 2400 4250 50  0001 C CNN
-	1    2400 4250
-	1    0    0    -1
-$EndComp
-$Comp
-L Mechanical:MountingHole_Pad H4
-U 1 1 5DBE575C
-P 3000 4150
-F 0 "H4" H 3100 4201 50  0000 L CNN
-F 1 "MountingHole" H 2800 4325 50  0000 L CNN
-F 2 "MountingHole:MountingHole_3.2mm_M3_Pad" H 3000 4150 50  0001 C CNN
-F 3 "~" H 3000 4150 50  0001 C CNN
-	1    3000 4150
-	1    0    0    -1
+L Device:Polyfuse_Small F1
+U 1 1 5DBEC73F
+P 1175 2600
+F 0 "F1" V 970 2600 50  0000 C CNN
+F 1 "Polyfuse" V 1061 2600 50  0000 C CNN
+F 2 "Fuse:Fuse_1812_4532Metric_Pad1.30x3.40mm_HandSolder" H 1225 2400 50  0001 L CNN
+F 3 "~" H 1175 2600 50  0001 C CNN
+	1    1175 2600
+	0    1    1    0
 $EndComp
+Wire Wire Line
+	875  2600 1075 2600
 $Comp
-L power:GND #PWR019
-U 1 1 5DBE5762
-P 3000 4250
-F 0 "#PWR019" H 3000 4000 50  0001 C CNN
-F 1 "GND" H 3005 4077 50  0000 C CNN
-F 2 "" H 3000 4250 50  0001 C CNN
-F 3 "" H 3000 4250 50  0001 C CNN
-	1    3000 4250
+L Switch:SW_SPST SW2
+U 1 1 5DBF0754
+P 1475 2600
+F 0 "SW2" H 1425 2700 50  0000 L CNN
+F 1 "SW" H 1425 2525 50  0000 L CNN
+F 2 "Connector_PinHeader_2.54mm:PinHeader_1x02_P2.54mm_Vertical" H 1475 2600 50  0001 C CNN
+F 3 "" H 1475 2600 50  0001 C CNN
+	1    1475 2600
 	1    0    0    -1
 $EndComp
-NoConn ~ 9875 5025
+Wire Wire Line
+	1675 2600 2050 2600
+Wire Wire Line
+	2050 2600 2325 2600
+Connection ~ 2050 2600
 $EndSCHEMATC

Commit message: TP4056
Parts:
- removed BT1: Battery, Connector_JST:JST_XH_B02B-XH-A_1x02_P2.50mm_Vertical, symbol Device:Battery
- removed H1, H2: MountingHole, MountingHole:MountingHole_3.2mm_M3_Pad, symbol Mechanical:MountingHole_Pad
- removed J3: USB_UART_OFF, Connector_PinHeader_2.54mm:PinHeader_1x01_P2.54mm_Vertical, symbol Connector_Generic:Conn_01x01
- removed J4: USB_UART_ON, Connector_PinHeader_2.54mm:PinHeader_1x01_P2.54mm_Vertical, symbol Connector_Generic:Conn_01x01
- added J3: USB_UART, Connector_PinHeader_2.54mm:PinHeader_1x02_P2.54mm_Vertical, symbol Connector_Generic:Conn_01x02
- added J4: PWR, Connector_PinHeader_2.54mm:PinHeader_1x02_P2.54mm_Vertical, symbol Connector_Generic:Conn_01x02
Connections:
- net labels added: OUT+, OUT-, PWR
- net labels removed: BATT
Other:
- note added: "Lipo \nTP4056\nCharging Board"
Changed lines of the file:
@@
 $EndComp
 $Comp
-L Device:Battery BT1
-U 1 1 5DBC220B
-P 875 2800
-F 0 "BT1" H 983 2846 50  0000 L CNN
-F 1 "Battery" H 983 2755 50  0000 L CNN
-F 2 "Connector_JST:JST_XH_B02B-XH-A_1x02_P2.50mm_Vertical" V 875 2860 50  0001 C CNN
-F 3 "~" V 875 2860 50  0001 C CNN
-	1    875  2800
-	1    0    0    -1
-$EndComp
-$Comp
 L Device:C_Small C3
 U 1 1 5DBC2404
@@
 	3350 2900 2625 2900
 Connection ~ 2625 2900
-Wire Wire Line
-	2625 2900 2625 3050
-Wire Wire Line
-	875  3000 875  3050
-Wire Wire Line
-	875  3050 2625 3050
-Connection ~ 2625 3050
-Wire Wire Line
-	2625 3050 2625 3125
 Text Label 1825 2600 0    50   ~ 0
-BATT
+PWR
 NoConn ~ 6025 4425
 Text GLabel 6025 4525 0    50   Input ~ 0
@@
 $EndComp
 Text Label 1500 825  0    50   ~ 0
-BATT
+PWR
 Wire Wire Line
 	1700 925  1700 825
@@
 Text Notes 3725 6675 0    50   ~ 0
 Connect the power pin \nof the USB to UART chip,\nwith a bodge wire, \nto either off or on.
-Text GLabel 3525 2600 2    50   Input ~ 0
+Text GLabel 4175 2600 2    50   Input ~ 0
 3V3
 Wire Wire Line
-	3350 2600 3525 2600
+	3350 2600 4175 2600
 Connection ~ 3350 2600
 Text GLabel 6025 4325 0    50   Input ~ 0
@@
 Wire Wire Line
 	5625 4625 5625 4650
-Text GLabel 4125 5750 2    50   Input ~ 0
+Text GLabel 4125 6025 2    50   Input ~ 0
 3V3
 Wire Notes Line
-	600  2075 3775 2075
+	600  2075 4425 2075
 Wire Notes Line
-	3775 2075 3775 3475
+	4425 2075 4425 3475
 Wire Notes Line
-	3775 3475 600  3475
+	4425 3475 600  3475
 Wire Notes Line
 	600  3475 600  2075
@@
 Text Notes 650  700  0    79   ~ 16
 Sensors
-$Comp
-L Connector_Generic:Conn_01x01 J3
-U 1 1 5DBC844A
-P 3925 6125
-F 0 "J3" H 3925 6000 50  0000 C CNN
-F 1 "USB_UART_OFF" H 3875 6250 50  0000 C CNN
-F 2 "Connector_PinHeader_2.54mm:PinHeader_1x01_P2.54mm_Vertical" H 3925 6125 50  0001 C CNN
-F 3 "~" H 3925 6125 50  0001 C CNN
-	1    3925 6125
-	-1   0    0    1
-$EndComp
 Wire Notes Line width 31 rgb(0, 194, 0)
 	3650 6750 3650 6125
@@
 	2675 6750 3650 6750
 $Comp
-L Connector_Generic:Conn_01x01 J4
-U 1 1 5DBCB146
-P 3925 5750
-F 0 "J4" H 3925 5625 50  0000 C CNN
-F 1 "USB_UART_ON" H 3900 5875 50  0000 C CNN
-F 2 "Connector_PinHeader_2.54mm:PinHeader_1x01_P2.54mm_Vertical" H 3925 5750 50  0001 C CNN
-F 3 "~" H 3925 5750 50  0001 C CNN
-	1    3925 5750
-	-1   0    0    1
-$EndComp
-$Comp
 L power:GND #PWR010
 U 1 1 5DBCB1FE
@@
 Text GLabel 9875 4925 2    50   Input ~ 0
 SOIL_6
-$Comp
-L Mechanical:MountingHole_Pad H1
-U 1 1 5DBE4537
-P 1200 4150
-F 0 "H1" H 1300 4201 50  0000 L CNN
-F 1 "MountingHole" H 1000 4325 50  0000 L CNN
-F 2 "MountingHole:MountingHole_3.2mm_M3_Pad" H 1200 4150 50  0001 C CNN
-F 3 "~" H 1200 4150 50  0001 C CNN
-	1    1200 4150
-	1    0    0    -1
-$EndComp
-$Comp
-L power:GND #PWR016
-U 1 1 5DBE45D3
-P 1200 4250
-F 0 "#PWR016" H 1200 4000 50  0001 C CNN
-F 1 "GND" H 1205 4077 50  0000 C CNN
-F 2 "" H 1200 4250 50  0001 C CNN
-F 3 "" H 1200 4250 50  0001 C CNN
-	1    1200 4250
-	1    0    0    -1
-$EndComp
-$Comp
-L Mechanical:MountingHole_Pad H2
-U 1 1 5DBE47CF
-P 1800 4150
-F 0 "H2" H 1900 4201 50  0000 L CNN
-F 1 "MountingHole" H 1600 4325 50  0000 L CNN
-F 2 "MountingHole:MountingHole_3.2mm_M3_Pad" H 1800 4150 50  0001 C CNN
-F 3 "~" H 1800 4150 50  0001 C CNN
-	1    1800 4150
-	1    0    0    -1
-$EndComp
-$Comp
-L power:GND #PWR017
-U 1 1 5DBE47D5
-P 1800 4250
-F 0 "#PWR017" H 1800 4000 50  0001 C CNN
-F 1 "GND" H 1805 4077 50  0000 C CNN
-F 2 "" H 1800 4250 50  0001 C CNN
-F 3 "" H 1800 4250 50  0001 C CNN
-	1    1800 4250
-	1    0    0    -1
-$EndComp
 NoConn ~ 9875 5025
 Text Label 5825 4725 0    50   ~ 0
-BATT
+PWR
 Wire Wire Line
 	6025 4725 5825 4725
@@
 	0    1    1    0
 $EndComp
-Wire Wire Line
-	875  2600 1075 2600
 $Comp
 L Switch:SW_SPST SW2
@@
 	2050 2600 2325 2600
 Connection ~ 2050 2600
+$Comp
+L Connector_Generic:Conn_01x02 J3
+U 1 1 5DBF3074
+P 3925 6125
+F 0 "J3" H 3900 6250 50  0000 L CNN
+F 1 "USB_UART" H 3725 5900 50  0000 L CNN
+F 2 "Connector_PinHeader_2.54mm:PinHeader_1x02_P2.54mm_Vertical" H 3925 6125 50  0001 C CNN
+F 3 "~" H 3925 6125 50  0001 C CNN
+	1    3925 6125
+	-1   0    0    1
+$EndComp
+$Comp
+L Connector_Generic:Conn_01x02 J4
+U 1 1 5DBF418E
+P 825 2950
+F 0 "J4" H 825 2675 50  0000 C CNN
+F 1 "PWR" H 825 2750 50  0000 C CNN
+F 2 "Connector_PinHeader_2.54mm:PinHeader_1x02_P2.54mm_Vertical" H 825 2950 50  0001 C CNN
+F 3 "~" H 825 2950 50  0001 C CNN
+	1    825  2950
+	-1   0    0    1
+$EndComp
+Wire Wire Line
+	2625 2900 2625 3125
+Text Notes 650  3275 0    50   ~ 0
+Lipo \nTP4056\nCharging Board
+Wire Wire Line
+	1075 2600 1025 2600
+Wire Wire Line
+	1025 2600 1025 2850
+Wire Wire Line
+	1025 2950 1025 3125
+Wire Wire Line
+	1025 3125 2625 3125
+Connection ~ 2625 3125
+Text Label 1025 2775 0    50   ~ 0
+OUT+
+Text Label 1025 3050 0    50   ~ 0
+OUT-
 $EndSCHEMATC

Commit message: Alternate LDO
Parts:
- added C5, C6: 1uF, Capacitor_SMD:C_0603_1608Metric_Pad1.05x0.95mm_HandSolder, symbol Device:C_Small
- added U4: MCP1703A-3302_SOT223, Package_TO_SOT_SMD:SOT-223-3_TabPin2, symbol Regulator_Linear:MCP1703A-3302_SOT223
- J4: footprint Connector_PinHeader_2.54mm:PinHeader_1x02_P2.54mm_Vertical -> tp4056:tp4056
Connections:
- net 3V3: now also C6.1, U4.3 (VO)
- net GND: now also C5.2, C6.2, U4.2 (GND)
- net PWR: now also C5.1, U4.1 (VI)
Other:
- note added: "Alternate LDO\nfor up to 16V input"
- moved on the sheet: C3, C4
Changed lines of the file:
@@
 L power:GND #PWR06
 U 1 1 5DBC1A3A
-P 2625 3125
-F 0 "#PWR06" H 2625 2875 50  0001 C CNN
-F 1 "GND" H 2630 2952 50  0000 C CNN
-F 2 "" H 2625 3125 50  0001 C CNN
-F 3 "" H 2625 3125 50  0001 C CNN
-	1    2625 3125
+P 2625 2900
+F 0 "#PWR06" H 2625 2650 50  0001 C CNN
+F 1 "GND" H 2630 2727 50  0000 C CNN
+F 2 "" H 2625 2900 50  0001 C CNN
+F 3 "" H 2625 2900 50  0001 C CNN
+	1    2625 2900
 	1    0    0    -1
 $EndComp
@@
 L Device:C_Small C3
 U 1 1 5DBC2404
-P 2050 2800
-F 0 "C3" H 2142 2846 50  0000 L CNN
-F 1 "1uF" H 2142 2755 50  0000 L CNN
-F 2 "Capacitor_SMD:C_0603_1608Metric_Pad1.05x0.95mm_HandSolder" H 2050 2800 50  0001 C CNN
-F 3 "~" H 2050 2800 50  0001 C CNN
-	1    2050 2800
+P 2150 2700
+F 0 "C3" H 2242 2746 50  0000 L CNN
+F 1 "1uF" H 2242 2655 50  0000 L CNN
+F 2 "Capacitor_SMD:C_0603_1608Metric_Pad1.05x0.95mm_HandSolder" H 2150 2700 50  0001 C CNN
+F 3 "~" H 2150 2700 50  0001 C CNN
+	1    2150 2700
 	1    0    0    -1
 $EndComp
@@
 L Device:C_Small C4
 U 1 1 5DBC2493
-P 3350 2800
-F 0 "C4" H 3442 2846 50  0000 L CNN
-F 1 "1uF" H 3442 2755 50  0000 L CNN
-F 2 "Capacitor_SMD:C_0603_1608Metric_Pad1.05x0.95mm_HandSolder" H 3350 2800 50  0001 C CNN
-F 3 "~" H 3350 2800 50  0001 C CNN
-	1    3350 2800
+P 3000 2700
+F 0 "C4" H 3092 2746 50  0000 L CNN
+F 1 "1uF" H 3092 2655 50  0000 L CNN
+F 2 "Capacitor_SMD:C_0603_1608Metric_Pad1.05x0.95mm_HandSolder" H 3000 2700 50  0001 C CNN
+F 3 "~" H 3000 2700 50  0001 C CNN
+	1    3000 2700
 	1    0    0    -1
 $EndComp
-Wire Wire Line
-	3350 2700 3350 2600
-Wire Wire Line
-	3350 2600 2925 2600
-Wire Wire Line
-	2050 2700 2050 2600
-Wire Wire Line
-	2050 2900 2625 2900
-Wire Wire Line
-	3350 2900 2625 2900
-Connection ~ 2625 2900
 Text Label 1825 2600 0    50   ~ 0
 PWR
@@
 Text GLabel 4175 2600 2    50   Input ~ 0
 3V3
-Wire Wire Line
-	3350 2600 4175 2600
-Connection ~ 3350 2600
 Text GLabel 6025 4325 0    50   Input ~ 0
 3V3
@@
 	600  2075 4425 2075
 Wire Notes Line
-	4425 2075 4425 3475
-Wire Notes Line
-	4425 3475 600  3475
-Wire Notes Line
-	600  3475 600  2075
+	4425 4075 600  4075
 Text Notes 650  2225 0    79   ~ 16
 Power
@@
 	1    0    0    -1
 $EndComp
-Wire Wire Line
-	1675 2600 2050 2600
-Wire Wire Line
-	2050 2600 2325 2600
-Connection ~ 2050 2600
 $Comp
 L Connector_Generic:Conn_01x02 J3
@@
 F 0 "J4" H 825 2675 50  0000 C CNN
 F 1 "PWR" H 825 2750 50  0000 C CNN
-F 2 "Connector_PinHeader_2.54mm:PinHeader_1x02_P2.54mm_Vertical" H 825 2950 50  0001 C CNN
+F 2 "tp4056:tp4056" H 825 2950 50  0001 C CNN
 F 3 "~" H 825 2950 50  0001 C CNN
 	1    825  2950
 	-1   0    0    1
 $EndComp
-Wire Wire Line
-	2625 2900 2625 3125
-Text Notes 650  3275 0    50   ~ 0
+Text Notes 625  3450 0    50   ~ 0
 Lipo \nTP4056\nCharging Board
 Wire Wire Line
@@
 Wire Wire Line
 	1025 2950 1025 3125
-Wire Wire Line
-	1025 3125 2625 3125
-Connection ~ 2625 3125
 Text Label 1025 2775 0    50   ~ 0
 OUT+
 Text Label 1025 3050 0    50   ~ 0
 OUT-
+$Comp
+L Regulator_Linear:MCP1703A-3302_SOT223 U4
+U 1 1 5DC182DA
+P 2625 3475
+F 0 "U4" H 2625 3717 50  0000 C CNN
+F 1 "MCP1703A-3302_SOT223" H 2625 3626 50  0000 C CNN
+F 2 "Package_TO_SOT_SMD:SOT-223-3_TabPin2" H 2625 3675 50  0001 C CNN
+F 3 "http://ww1.microchip.com/downloads/en/DeviceDoc/20005122B.pdf" H 2625 3425 50  0001 C CNN
+	1    2625 3475
+	1    0    0    -1
+$EndComp
+Wire Wire Line
+	2325 3475 2175 3475
+Wire Wire Line
+	2925 3475 3025 3475
+$Comp
+L power:GND #PWR016
+U 1 1 5DC1D21C
+P 2625 3775
+F 0 "#PWR016" H 2625 3525 50  0001 C CNN
+F 1 "GND" H 2630 3602 50  0000 C CNN
+F 2 "" H 2625 3775 50  0001 C CNN
+F 3 "" H 2625 3775 50  0001 C CNN
+	1    2625 3775
+	1    0    0    -1
+$EndComp
+$Comp
+L power:GND #PWR015
+U 1 1 5DC1E5D1
+P 1025 3125
+F 0 "#PWR015" H 1025 2875 50  0001 C CNN
+F 1 "GND" H 1030 2952 50  0000 C CNN
+F 2 "" H 1025 3125 50  0001 C CNN
+F 3 "" H 1025 3125 50  0001 C CNN
+	1    1025 3125
+	1    0    0    -1
+$EndComp
+Wire Notes Line
+	600  2075 600  4075
+Wire Notes Line
+	4425 2075 4425 4075
+Connection ~ 3000 2600
+Wire Wire Line
+	3000 2600 2925 2600
+Connection ~ 2150 2600
+Wire Wire Line
+	2150 2600 2325 2600
+Wire Wire Line
+	1675 2600 1775 2600
+Wire Wire Line
+	3000 2600 3350 2600
+Wire Wire Line
+	2150 2800 2150 2900
+Wire Wire Line
+	2150 2900 2625 2900
+Connection ~ 2625 2900
+Wire Wire Line
+	2625 2900 3000 2900
+Wire Wire Line
+	3000 2900 3000 2800
+$Comp
+L Device:C_Small C5
+U 1 1 5DC24C67
+P 2175 3575
+F 0 "C5" H 2267 3621 50  0000 L CNN
+F 1 "1uF" H 2267 3530 50  0000 L CNN
+F 2 "Capacitor_SMD:C_0603_1608Metric_Pad1.05x0.95mm_HandSolder" H 2175 3575 50  0001 C CNN
+F 3 "~" H 2175 3575 50  0001 C CNN
+	1    2175 3575
+	1    0    0    -1
+$EndComp
+Connection ~ 2175 3475
+$Comp
+L Device:C_Small C6
+U 1 1 5DC24CF9
+P 3025 3575
+F 0 "C6" H 3117 3621 50  0000 L CNN
+F 1 "1uF" H 3117 3530 50  0000 L CNN
+F 2 "Capacitor_SMD:C_0603_1608Metric_Pad1.05x0.95mm_HandSolder" H 3025 3575 50  0001 C CNN
+F 3 "~" H 3025 3575 50  0001 C CNN
+	1    3025 3575
+	1    0    0    -1
+$EndComp
+Connection ~ 3025 3475
+Wire Wire Line
+	3025 3475 3350 3475
+Wire Wire Line
+	2175 3675 2175 3775
+Wire Wire Line
+	2175 3775 2625 3775
+Connection ~ 2625 3775
+Wire Wire Line
+	2625 3775 3025 3775
+Wire Wire Line
+	3025 3775 3025 3675
+Wire Wire Line
+	1775 3475 1775 2600
+Wire Wire Line
+	1775 3475 2175 3475
+Connection ~ 1775 2600
+Wire Wire Line
+	1775 2600 2150 2600
+Wire Wire Line
+	3350 3475 3350 2600
+Connection ~ 3350 2600
+Wire Wire Line
+	3350 2600 4175 2600
+Text Notes 2800 3975 0    50   ~ 0
+Alternate LDO\nfor up to 16V input
+Wire Notes Line
+	1600 4075 1600 3150
+Wire Notes Line
+	1600 3150 3775 3150
+Wire Notes Line
+	3775 3150 3775 4075
 $EndSCHEMATC
