File: receiver/hardware/kicad/receiver/receiver.sch (KiCad schematic (older format))
At the start: 27 parts, among them J1 Connector, U1 74HC595, U2 74HC595

Commit message: Initial layout
Parts:
- D1, D2, D4, D5, D7: footprint LED_THT:LED_D5.0mm-4_RGB_Wide_Pins -> LED_THT:LED_D5.0mm-4_RGB_Staggered_Pins
Connections:
- net at R25.2: now also U2.15 (QA)
- net at U2.1 (QB): now also R4.2; no longer R7.2
- net at U2.2 (QC): now also R7.2; no longer R10.2
- net at U2.3 (QD): now also R10.2; no longer R13.2
- net at U2.4 (QE): now also R13.2; no longer R16.2
- net at U2.5 (QF): now also R16.2; no longer R19.2
- net at U2.6 (QG): now also R19.2
- no-connect marks 4 -> 3
Other:
- moved on the sheet: D5, R13, R16, R19
Changed lines of the file:
@@
 F 0 "D1" H 4875 3750 50  0000 R CNN
 F 1 "RGB" H 4900 3000 50  0000 R CNN
-F 2 "LED_THT:LED_D5.0mm-4_RGB_Wide_Pins" H 4825 3300 50  0001 C CNN
+F 2 "LED_THT:LED_D5.0mm-4_RGB_Staggered_Pins" H 4825 3300 50  0001 C CNN
 F 3 "~" H 4825 3300 50  0001 C CNN
 	1    4825 3350
@@
 F 0 "D4" H 4875 4700 50  0000 R CNN
 F 1 "RGB" H 4900 3950 50  0000 R CNN
-F 2 "LED_THT:LED_D5.0mm-4_RGB_Wide_Pins" H 4825 4250 50  0001 C CNN
+F 2 "LED_THT:LED_D5.0mm-4_RGB_Staggered_Pins" H 4825 4250 50  0001 C CNN
 F 3 "~" H 4825 4250 50  0001 C CNN
 	1    4825 4300
@@
 F 0 "D7" H 4875 5650 50  0000 R CNN
 F 1 "RGB" H 4900 4900 50  0000 R CNN
-F 2 "LED_THT:LED_D5.0mm-4_RGB_Wide_Pins" H 4825 5200 50  0001 C CNN
+F 2 "LED_THT:LED_D5.0mm-4_RGB_Staggered_Pins" H 4825 5200 50  0001 C CNN
 F 3 "~" H 4825 5200 50  0001 C CNN
 	1    4825 5250
@@
 F 0 "D2" H 8450 3875 50  0000 R CNN
 F 1 "RGB" H 8475 3125 50  0000 R CNN
-F 2 "LED_THT:LED_D5.0mm-4_RGB_Wide_Pins" H 8400 3425 50  0001 C CNN
+F 2 "LED_THT:LED_D5.0mm-4_RGB_Staggered_Pins" H 8400 3425 50  0001 C CNN
 F 3 "~" H 8400 3425 50  0001 C CNN
 	1    8400 3475
@@
 L Device:LED_CRGB D5
 U 1 1 5E1C45F4
-P 8400 4425
-F 0 "D5" H 8450 4825 50  0000 R CNN
-F 1 "RGB" H 8475 4075 50  0000 R CNN
-F 2 "LED_THT:LED_D5.0mm-4_RGB_Wide_Pins" H 8400 4375 50  0001 C CNN
-F 3 "~" H 8400 4375 50  0001 C CNN
-	1    8400 4425
+P 8400 4625
+F 0 "D5" H 8450 5025 50  0000 R CNN
+F 1 "RGB" H 8475 4275 50  0000 R CNN
+F 2 "LED_THT:LED_D5.0mm-4_RGB_Staggered_Pins" H 8400 4575 50  0001 C CNN
+F 3 "~" H 8400 4575 50  0001 C CNN
+	1    8400 4625
 	-1   0    0    -1
 $EndComp
@@
 L Device:R R19
 U 1 1 5E1C45FB
+P 8050 4825
+F 0 "R19" V 8150 4825 50  0000 C CNN
+F 1 "1K" V 8050 4825 50  0000 C CNN
+F 2 "Resistor_SMD:R_0603_1608Metric_Pad1.05x0.95mm_HandSolder" V 7980 4825 50  0001 C CNN
+F 3 "~" H 8050 4825 50  0001 C CNN
+	1    8050 4825
+	0    1    1    0
+$EndComp
+$Comp
+L Device:R R16
+U 1 1 5E1C4602
 P 8050 4625
-F 0 "R19" V 8150 4625 50  0000 C CNN
+F 0 "R16" V 8150 4625 50  0000 C CNN
 F 1 "1K" V 8050 4625 50  0000 C CNN
 F 2 "Resistor_SMD:R_0603_1608Metric_Pad1.05x0.95mm_HandSolder" V 7980 4625 50  0001 C CNN
@@
 $EndComp
 $Comp
-L Device:R R16
-U 1 1 5E1C4602
+L Device:R R13
+U 1 1 5E1C4609
 P 8050 4425
-F 0 "R16" V 8150 4425 50  0000 C CNN
+F 0 "R13" V 8150 4425 50  0000 C CNN
 F 1 "1K" V 8050 4425 50  0000 C CNN
 F 2 "Resistor_SMD:R_0603_1608Metric_Pad1.05x0.95mm_HandSolder" V 7980 4425 50  0001 C CNN
@@
 	0    1    1    0
 $EndComp
-$Comp
-L Device:R R13
-U 1 1 5E1C4609
-P 8050 4225
-F 0 "R13" V 8150 4225 50  0000 C CNN
-F 1 "1K" V 8050 4225 50  0000 C CNN
-F 2 "Resistor_SMD:R_0603_1608Metric_Pad1.05x0.95mm_HandSolder" V 7980 4225 50  0001 C CNN
-F 3 "~" H 8050 4225 50  0001 C CNN
-	1    8050 4225
-	0    1    1    0
-$EndComp
-Wire Wire Line
-	6975 4425 7900 4425
-Wire Wire Line
-	6975 4325 7900 4325
-Wire Wire Line
-	7900 4325 7900 4225
-Wire Wire Line
-	6975 4225 7800 4225
-Wire Wire Line
-	7800 4225 7800 3675
-Wire Wire Line
-	7800 3675 7900 3675
-Wire Wire Line
-	6975 4125 7700 4125
-Wire Wire Line
-	7700 4125 7700 3475
-Wire Wire Line
-	7700 3475 7900 3475
-Wire Wire Line
-	6975 4025 7600 4025
-Wire Wire Line
-	7600 4025 7600 3275
-Wire Wire Line
-	7600 3275 7900 3275
-Wire Wire Line
-	6975 4525 7900 4525
-Wire Wire Line
-	7900 4525 7900 4625
+Wire Wire Line
+	7775 3675 7900 3675
+Wire Wire Line
+	7650 3475 7900 3475
 $Comp
 L Device:C_Small C2
@@
 L power:GND #PWR018
 U 1 1 5E1C4674
-P 8725 4425
-F 0 "#PWR018" H 8725 4175 50  0001 C CNN
-F 1 "GND" H 8730 4252 50  0000 C CNN
-F 2 "" H 8725 4425 50  0001 C CNN
-F 3 "" H 8725 4425 50  0001 C CNN
-	1    8725 4425
-	1    0    0    -1
-$EndComp
-Wire Wire Line
-	8600 4425 8725 4425
-Wire Wire Line
-	6175 4025 5400 4025
-Wire Wire Line
-	5400 4025 5400 6150
-Wire Wire Line
-	5400 6150 3400 6150
+P 8725 4625
+F 0 "#PWR018" H 8725 4375 50  0001 C CNN
+F 1 "GND" H 8730 4452 50  0000 C CNN
+F 2 "" H 8725 4625 50  0001 C CNN
+F 3 "" H 8725 4625 50  0001 C CNN
+	1    8725 4625
+	1    0    0    -1
+$EndComp
+Wire Wire Line
+	8600 4625 8725 4625
+Wire Wire Line
+	6175 4025 5500 4025
+Wire Wire Line
+	5500 4025 5500 6150
+Wire Wire Line
+	5500 6150 3400 6150
 Wire Wire Line
 	3400 6150 3400 4800
@@
 LDR
 NoConn ~ 4375 2025
-NoConn ~ 6975 4625
 NoConn ~ 6975 4725
 NoConn ~ 6975 4925
+Wire Wire Line
+	6975 4025 7425 4025
+Wire Wire Line
+	7425 4025 7425 3050
+Wire Wire Line
+	7425 3050 5325 3050
+Wire Wire Line
+	5325 3050 5325 5750
+Wire Wire Line
+	5325 5750 4325 5750
+Wire Wire Line
+	4325 5750 4325 5450
+Wire Wire Line
+	6975 4125 7550 4125
+Wire Wire Line
+	7550 4125 7550 3275
+Wire Wire Line
+	7550 3275 7900 3275
+Wire Wire Line
+	6975 4225 7650 4225
+Wire Wire Line
+	7650 4225 7650 3475
+Wire Wire Line
+	6975 4325 7775 4325
+Wire Wire Line
+	7775 4325 7775 3675
+Wire Wire Line
+	6975 4425 7900 4425
+Wire Wire Line
+	6975 4525 7775 4525
+Wire Wire Line
+	7775 4525 7775 4625
+Wire Wire Line
+	7775 4625 7900 4625
+Wire Wire Line
+	6975 4625 7675 4625
+Wire Wire Line
+	7675 4625 7675 4825
+Wire Wire Line
+	7675 4825 7900 4825
 $EndSCHEMATC

Commit message: Wired
Parts:
- D1, D2, D4, D5, D7: footprint LED_THT:LED_D5.0mm-4_RGB_Staggered_Pins -> LED_THT:LED_D5.0mm-4_RGB; symbol Device:LED_CRGB -> Device:LED_RCGB
Connections:
- net GND: now also D1.2 (K), D2.2 (K), D4.2 (K), D5.2 (K), D7.2 (K); no longer D1.1 (K), D2.1 (K), D4.1 (K), D5.1 (K), D7.1 (K)
- net at R3.1: now also D1.1 (RA); no longer D1.2 (RA)
- net at R12.1: now also D4.1 (RA); no longer D4.2 (RA)
- net at R21.1: now also D7.1 (RA); no longer D7.2 (RA)
- net at R4.1: now also D2.1 (RA); no longer D2.2 (RA)
- net at R13.1: now also D5.1 (RA); no longer D5.2 (RA)
Changed lines of the file:
@@
 $EndDescr
 $Comp
-L Device:LED_CRGB D1
+L Device:LED_RCGB D1
 U 1 1 5E1B5456
 P 4825 3350
 F 0 "D1" H 4875 3750 50  0000 R CNN
 F 1 "RGB" H 4900 3000 50  0000 R CNN
-F 2 "LED_THT:LED_D5.0mm-4_RGB_Staggered_Pins" H 4825 3300 50  0001 C CNN
+F 2 "LED_THT:LED_D5.0mm-4_RGB" H 4825 3300 50  0001 C CNN
 F 3 "~" H 4825 3300 50  0001 C CNN
 	1    4825 3350
@@
 $EndComp
 $Comp
-L Device:LED_CRGB D4
+L Device:LED_RCGB D4
 U 1 1 5E1B6E70
 P 4825 4300
 F 0 "D4" H 4875 4700 50  0000 R CNN
 F 1 "RGB" H 4900 3950 50  0000 R CNN
-F 2 "LED_THT:LED_D5.0mm-4_RGB_Staggered_Pins" H 4825 4250 50  0001 C CNN
+F 2 "LED_THT:LED_D5.0mm-4_RGB" H 4825 4250 50  0001 C CNN
 F 3 "~" H 4825 4250 50  0001 C CNN
 	1    4825 4300
@@
 $EndComp
 $Comp
-L Device:LED_CRGB D7
+L Device:LED_RCGB D7
 U 1 1 5E1B7049
 P 4825 5250
 F 0 "D7" H 4875 5650 50  0000 R CNN
 F 1 "RGB" H 4900 4900 50  0000 R CNN
-F 2 "LED_THT:LED_D5.0mm-4_RGB_Staggered_Pins" H 4825 5200 50  0001 C CNN
+F 2 "LED_THT:LED_D5.0mm-4_RGB" H 4825 5200 50  0001 C CNN
 F 3 "~" H 4825 5200 50  0001 C CNN
 	1    4825 5250
@@
 	5025 5250 5150 5250
 $Comp
-L Device:LED_CRGB D2
+L Device:LED_RCGB D2
 U 1 1 5E1C45CB
 P 8400 3475
 F 0 "D2" H 8450 3875 50  0000 R CNN
 F 1 "RGB" H 8475 3125 50  0000 R CNN
-F 2 "LED_THT:LED_D5.0mm-4_RGB_Staggered_Pins" H 8400 3425 50  0001 C CNN
+F 2 "LED_THT:LED_D5.0mm-4_RGB" H 8400 3425 50  0001 C CNN
 F 3 "~" H 8400 3425 50  0001 C CNN
 	1    8400 3475
@@
 $EndComp
 $Comp
-L Device:LED_CRGB D5
+L Device:LED_RCGB D5
 U 1 1 5E1C45F4
 P 8400 4625
 F 0 "D5" H 8450 5025 50  0000 R CNN
 F 1 "RGB" H 8475 4275 50  0000 R CNN
-F 2 "LED_THT:LED_D5.0mm-4_RGB_Staggered_Pins" H 8400 4575 50  0001 C CNN
+F 2 "LED_THT:LED_D5.0mm-4_RGB" H 8400 4575 50  0001 C CNN
 F 3 "~" H 8400 4575 50  0001 C CNN
 	1    8400 4625
@@
 Wire Wire Line
 	7675 4825 7900 4825
+Text Label 5725 4325 0    50   ~ 0
+RST
+Text Label 2125 4200 0    50   ~ 0
+RST
 $EndSCHEMATC
